File: Grub Compass PCB/Grub Compass.kicad_pcb (KiCad board)
At the start: 2 copper layers, 23 parts, among them Q1 IRLML6302TRPBF, SW1 TS-1088-AR02016, SW2 TS-1088-AR02016, U2 AMS1117-3.3, U4 MCP73831-2-OT, U6 ESP32-WROOM-32E

Commit message: PCB Day 3
Parts:
- added BatteryConnector1: Conn_01x02_Pin, grubCompass:PinHeader_1x02_P1.00mm_Vertical, F.Cu at (131.0, 123.0)
- added CONN_HDR_3POS_1612901-1: Conn_01x03_Pin, Connector_PinHeader_1.00mm:PinHeader_1x03_P1.00mm_Vertical, F.Cu at (113.5, 121.0)
- added D4: 1N5819, Diode_SMD:D_SOD-123, F.Cu at (109.5, 105.7)
- added D5: 1N5819, Diode_SMD:D_SOD-123, F.Cu at (109.5, 109.0)
- added GPS_Connector1: Conn_01x04_Pin, Connector_PinHeader_1.00mm:PinHeader_1x04_P1.00mm_Vertical, F.Cu at (186.5, 116.0)
- added IMU_Connector1: Conn_01x04_Pin, Connector_PinHeader_1.00mm:PinHeader_1x04_P1.00mm_Vertical, F.Cu at (173.5, 119.0)
- added J1: USB_C_Receptacle_USB2.0_16P, Connector_USB:USB_C_Receptacle_G-Switch_GT-USB-7010ASV, F.Cu at (150.0, 136.0)
- added J2: Conn_01x08_Pin, Connector_PinHeader_1.00mm:PinHeader_1x08_P1.00mm_Vertical, F.Cu at (163.0, 106.5)
- added R10: 10K, Resistor_SMD:R_1206_3216Metric, F.Cu at (166.5, 115.5)
- added R4: 5.1k, PCM_JLCPCB:R_0603, F.Cu at (114.2, 111.8)
- added R5: 5.1k, PCM_JLCPCB:R_0603, F.Cu at (114.2, 114.0)
- added R9: 10K, Resistor_SMD:R_1206_3216Metric, F.Cu at (115.2, 105.7)
- added SERVO_Connector1: Conn_01x03_Pin, Connector_PinHeader_1.00mm:PinHeader_1x03_P1.00mm_Vertical, F.Cu at (201.0, 117.0)
- added U3: BC-4-3PD, grubCompass:BC-4-3PD, F.Cu at (113.0, 97.0)
- moved D2 53.6 mm to (188.0, 153.8)
- moved Q1 41.9 mm to (194.1, 149.3)
- moved C2 35.5 mm to (183.8, 143.6)
- moved C6 35.5 mm to (199.8, 140.7)
- moved D3 35.5 mm to (173.7, 141.3)
- moved U4 35.5 mm to (188.6, 141.4)
- moved C1 35.5 mm to (183.8, 140.5)
- moved C3 35.5 mm to (175.5, 144.6)
- moved C4 35.5 mm to (179.6, 140.2)
- moved C5 35.5 mm to (175.5, 146.5)
- moved C7 35.5 mm to (179.6, 142.4)
- moved C8 35.5 mm to (179.6, 144.7)
- moved R1 35.5 mm to (201.7, 143.3)
- moved R2 35.5 mm to (201.7, 145.0)
- moved R3 35.5 mm to (201.7, 146.8)
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- renumbered SW1 to BOOT, SW2 to EN
Connections:
- net Net-(D1-K) renamed SERVO_5V
- U6 pad 14: BAT_MEAS -> Net-(U6-IO12)
- U6 pad 24: unconnected-(U6-IO2-Pad24) -> Net-(U6-IO2)
- U6 pad 26: unconnected-(U6-IO4-Pad26) -> Net-(J2-Pin_3)
- U6 pad 28: unconnected-(U6-IO17-Pad28) -> Net-(J2-Pin_5)
- U6 pad 29: unconnected-(U6-IO5-Pad29) -> Net-(J2-Pin_4)
- U6 pad 30: unconnected-(U6-IO18-Pad30) -> Net-(J2-Pin_6)
- U6 pad 31: SERVO_PWM -> Net-(J2-Pin_7)
- U6 pad 33: unconnected-(U6-IO21-Pad33) -> SDA
- U6 pad 36: unconnected-(U6-IO22-Pad36) -> SCL
- U6 pad 37: unconnected-(U6-IO23-Pad37) -> Net-(J2-Pin_8)
- U6 pad 7: unconnected-(U6-IO35-Pad7) -> BAT_MEAS
Other:
- board outline added: 29 x 59 mm

Commit message: Breaking more things
Parts:
- removed BatteryConnector1: Conn_01x02_Pin, grubCompass:PinHeader_1x02_P1.00mm_Vertical
- removed CONN_HDR_3POS_1612901-1, SERVO_Connector1: Conn_01x03_Pin, Connector_PinHeader_1.00mm:PinHeader_1x03_P1.00mm_Vertical
- removed GPS_Connector1, IMU_Connector1: Conn_01x04_Pin, Connector_PinHeader_1.00mm:PinHeader_1x04_P1.00mm_Vertical
- removed U3: BC-4-3PD, grubCompass:BC-4-3PD
- added Battery: Conn_01x02_Pin, grubCompass:PinHeader_1x02_P1.00mm_Vertical, F.Cu at (163.0, 97.2)
- added DOCK: Conn_01x03_Pin, Connector_PinHeader_1.00mm:PinHeader_1x03_P1.00mm_Vertical, F.Cu at (136.8, 106.0)
- added GPS: Conn_01x04_Pin, Connector_PinHeader_1.00mm:PinHeader_1x04_P1.00mm_Vertical, F.Cu at (136.8, 95.0)
- added IMU: Conn_01x04_Pin, Connector_PinHeader_1.00mm:PinHeader_1x04_P1.00mm_Vertical, F.Cu at (136.8, 97.0)
- added SERVO: Conn_01x03_Pin, Connector_PinHeader_1.00mm:PinHeader_1x03_P1.00mm_Vertical, F.Cu at (136.8, 102.0)
- moved R6 58.9 mm to (139.0, 123.0)
- moved C6 57.1 mm to (147.0, 119.0)
- moved R1 55.3 mm to (156.0, 112.0)
- moved D5 53.3 mm to (158.0, 131.0)
- moved Q1 50.5 mm to (157.0, 115.0)
- moved R3 49.2 mm to (158.0, 124.0)
- moved C2 46.0 mm to (147.0, 116.0)
- moved R2 44.6 mm to (160.0, 129.0)
- moved D4 44.3 mm to (152.0, 118.0)
- moved D1 42.9 mm to (157.0, 119.0)
- moved R8 42.8 mm to (153.0, 124.0), turned to -90 degrees
- moved D2 41.7 mm to (156.0, 127.0), turned to -90 degrees
- moved R4 41.1 mm to (151.0, 130.0)
- moved R5 40.0 mm to (152.0, 127.0)
- moved R7 39.2 mm to (163.0, 127.0)
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Connections:
- U6 pad 13: unconnected-(U6-IO14-Pad13) -> SERVO_PWM
- U6 pad 28: Net-(J2-Pin_5) -> Net-(J2-Pin_4)
- U6 pad 29: Net-(J2-Pin_4) -> Net-(J2-Pin_5)
Routing:
- net GND: track 0.00 -> 130.7 mm, vias 0 -> 9
- net BAT_MEAS: track 0.00 -> 89.2 mm
- net SERVO_5V: track 0.00 -> 70.8 mm, vias 0 -> 1
- net +3.3V: track 0.00 -> 45.5 mm
- net USB_5V: track 0.00 -> 43.0 mm, vias 0 -> 4
- net BAT+: track 0.00 -> 39.4 mm, vias 0 -> 3
- net USB_D-: track 0.00 -> 34.7 mm, vias 0 -> 2
- net +3V3: track 0.00 -> 33.6 mm, vias 0 -> 1
- net SDA: track 0.00 -> 29.8 mm, vias 0 -> 2
- net SCL: track 0.00 -> 28.4 mm, vias 0 -> 1
- net USB_D+: track 0.00 -> 27.7 mm, vias 0 -> 2
- net Net-(CONN_HDR_3POS_1612901-1-Pin_1): track 0.00 -> 21.9 mm
- net BOOT: track 0.00 -> 20.5 mm
- net Net-(U4-STAT): track 0.00 -> 18.7 mm, vias 0 -> 2
- net EN: track 0.00 -> 17.8 mm
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Other:
- board size 29 x 59 mm -> 32.5 x 59 mm
- board text added: "Badly designed by Milan B. Mishra on 6/7/2025"
