File: Grub Compass PCB/Grub Compass.kicad_sch (KiCad schematic)
At the start: 28 parts, among them J1 USB_C_Receptacle_USB2.0_16P, M1 Motor_Servo, Q1 IRLML6302TRPBF, SW1 TS-1088-AR02016, SW2 TS-1088-AR02016, U1 ESP32-C3-WROOM-02, U2 AMS1117-3.3, U3 BC-4-3PD, U4 MCP73831-2-OT

Commit message: Day 3 update
Parts:
- removed J1: USB_C_Receptacle_USB2.0_16P, symbol Connector:USB_C_Receptacle_USB2.0_16P
- removed R4, R5: 5.1k, Resistor_SMD:R_0201_0603Metric, symbol Device:R
- removed U1: ESP32-C3-WROOM-02, RF_Module:ESP32-C3-WROOM-02, symbol RF_Module:ESP32-C3-WROOM-02
- added U1: CONN_HDR_3POS_1612901-1, symbol grubCompass:CONN_HDR_3POS_1612898-1
- added U5: ~, symbol grubCompass:MINI_GPS_PA1010D_STEMMA_QT
- added U6: ESP32-WROOM-32E, RF_Module:ESP32-WROOM-32D, symbol RF_Module:ESP32-WROOM-32E
Connections:
- net +3.3V: now also M1.2 (+), U5.7 (VIN)
- net +3V3: now also U6.2 (VDD)
- net BAT_MEAS: now also U6.14 (IO12)
- net BOOT: now also U6.25 (IO0)
- net EN: now also U6.3 (EN)
- net GND: now also U1.3 (GND), U5.9 (GND), U6.1 (GND), U6.15 (GND), U6.38 (GND), U6.39 (GND)
- net USB_5V: now also U1.1 (5V)
- net USB_D+: now also U6.23 (IO15)
- net USB_D-: now also U6.27 (IO16)
- net SERVO renamed SERVO_PWM
- net SERVO_PWM: now also U6.31 (IO19)
- new net GPS_SDA: U5.11 (SDA)
- new net GPS_SDL: U5.10 (SCL)
- no-connect marks 3 -> 10
Other:
- note added: "Female Power Connector"
- note added: "MINI GPS PA1010D"
- note added: "Magnetometer"
- note added: "Servo"
- note removed: "USB Type-C Connector"
- moved on the sheet: M1, R3, SW1

Commit message: Day 4ish
Other:
- note added: "IMU"
- note removed: "Magnetometer"
Changed lines of the file:
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@@
 		(stroke
 			(width 0)
-			(type default)
+			(type solid)
 		)
 		(fill
@@
 		)
 	)
-	(text "Magnetometer"
+	(text "IMU"
 		(exclude_from_sim no)
 		(at 187.452 149.098 0)

Commit message: PCB Day 3
Parts:
- removed M1: Motor_Servo, symbol Motor:Motor_Servo
- removed U1: CONN_HDR_3POS_1612901-1, symbol grubCompass:CONN_HDR_3POS_1612898-1
- removed U3: BC-4-3PD, symbol grubCompass:BC-4-3PD
- removed U5: ~, symbol grubCompass:MINI_GPS_PA1010D_STEMMA_QT
- added BatteryConnector1: Conn_01x02_Pin, grubCompass:PinHeader_1x02_P1.00mm_Vertical, symbol Connector:Conn_01x02_Pin
- added CONN_HDR_3POS_1612901-1, SERVO_Connector1: Conn_01x03_Pin, Connector_PinHeader_1.00mm:PinHeader_1x03_P1.00mm_Vertical, symbol Connector:Conn_01x03_Pin
- added D4, D5: 1N5819, Diode_SMD:D_SOD-123, symbol Diode:1N5819
- added GPS_Connector1, IMU_Connector1: Conn_01x04_Pin, Connector_PinHeader_1.00mm:PinHeader_1x04_P1.00mm_Vertical, symbol Connector:Conn_01x04_Pin
- added J1: USB_C_Receptacle_USB2.0_16P, Connector_USB:USB_C_Receptacle_G-Switch_GT-USB-7010ASV, symbol Connector:USB_C_Receptacle_USB2.0_16P
- added J2: Conn_01x08_Pin, Connector_PinHeader_1.00mm:PinHeader_1x08_P1.00mm_Vertical, symbol Connector:Conn_01x08_Pin
- added R10, R9: 10K, Resistor_SMD:R_1206_3216Metric, symbol Device:R
- added R4, R5: 5.1k, PCM_JLCPCB:R_0603, symbol Device:R
Connections:
- net +3.3V: now also GPS_Connector1.4 (Pin_4), IMU_Connector1.1 (Pin_1)
- net +3V3: now also J2.1 (Pin_1)
- net BAT+: now also BatteryConnector1.2 (BAT+)
- net BAT_MEAS: now also U6.7 (IO35); no longer U6.14 (IO12)
- net GND: now also BatteryConnector1.1 (GND), CONN_HDR_3POS_1612901-1.3 (Pin_3), GPS_Connector1.3 (Pin_3), IMU_Connector1.2 (Pin_2), J1.A1 (GND), J1.A12 (GND), J1.B1 (GND), J1.B12 (GND), J1.S1 (SHIELD), J2.2 (Pin_2), R10.2, R4.2, R5.2, R9.2, SERVO_Connector1.1 (Pin_1)
- net SERVO_5V: now also C1.1, D1.1 (K), Q1.3 (S), U2.3 (VI), SERVO_Connector1.2 (Pin_2)
- net SERVO_PWM: now also SERVO_Connector1.3 (Pin_3); no longer U6.31 (IO19)
- net USB_5V: now also D4.1 (K), D5.1 (K)
- net USB_D+: now also J1.A6 (D+), J1.B6 (D+)
- net USB_D-: now also J1.A7 (D-), J1.B7 (D-)
- net at U6.24 (IO2): now also R10.1
- net at U6.26 (IO4): now also J2.3 (Pin_3)
- net at U6.28 (IO17): now also J2.5 (Pin_5)
- net at U6.29 (IO5): now also J2.4 (Pin_4)
- net at U6.30 (IO18): now also J2.6 (Pin_6)
- net SDA: now reaches U6.33 (IO21)
- net SDA: now also GPS_Connector1.1 (Pin_1), IMU_Connector1.4 (Pin_4)
- net SCL: now reaches U6.36 (IO22)
- net SCL: now also GPS_Connector1.2 (Pin_2), IMU_Connector1.3 (Pin_3)
- net at U6.37 (IO23): now also J2.8 (Pin_8)
- new net: R9.1, U6.14 (IO12)
- new net: J1.B5 (CC2), R5.1
- new net: J2.7 (Pin_7), U6.31 (IO19)
- new net: J1.A5 (CC1), R4.1
- new net: CONN_HDR_3POS_1612901-1.1 (Pin_1), D4.2 (A)
- new net: D5.2 (A), J1.A4 (VBUS), J1.A9 (VBUS), J1.B4 (VBUS), J1.B9 (VBUS)
- no-connect marks 10 -> 9
Other:
- note added: "Female Power Connector + USB-C"
- note removed: "Female Power Connector"
- moved on the sheet: U6

Commit message: Breaking more things
Connections:
- net SERVO_PWM: now also U6.13 (IO14)
- net at J2.4 (Pin_4): now also U6.28 (IO17); no longer U6.29 (IO5)
- net at J2.5 (Pin_5): now also U6.29 (IO5); no longer U6.28 (IO17)
- no-connect marks 9 -> 10
Changed lines of the file:
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@@
+	)
+	(no_connect
+		(at 116.84 59.69)
 	)
 	(no_connect
@@
 	(wire
 		(pts
-			(xy 106.68 59.69) (xy 116.84 59.69)
+			(xy 106.68 59.69) (xy 118.11 59.69)
 		)
 		(stroke
@@
 	(wire
 		(pts
+			(xy 116.84 44.45) (xy 106.68 44.45)
+		)
+		(stroke
+			(width 0)
+			(type default)
+		)
+	)
+	(wire
+		(pts
 			(xy 120.65 97.79) (xy 120.65 62.23)
 		)
@@
 	(wire
 		(pts
+			(xy 118.11 67.31) (xy 118.11 59.69)
+		)
+		(stroke
+			(width 0)
+			(type default)
+		)
+	)
+	(wire
+		(pts
 			(xy 106.68 72.39) (xy 113.03 72.39)
 		)
@@
 	(wire
 		(pts
-			(xy 116.84 69.85) (xy 116.84 59.69)
-		)
-		(stroke
-			(width 0)
-			(type default)
-		)
-	)
-	(wire
-		(pts
 			(xy 106.68 41.91) (xy 119.38 41.91)
 		)
@@
 	(wire
 		(pts
+			(xy 116.84 69.85) (xy 116.84 44.45)
+		)
+		(stroke
+			(width 0)
+			(type default)
+		)
+	)
+	(wire
+		(pts
 			(xy 160.02 229.87) (xy 170.18 229.87)
 		)
@@
 	(wire
 		(pts
-			(xy 118.11 44.45) (xy 118.11 67.31)
-		)
-		(stroke
-			(width 0)
-			(type default)
-		)
-	)
-	(wire
-		(pts
 			(xy 43.18 152.4) (xy 59.69 152.4)
 		)
@@
 	(wire
 		(pts
-			(xy 106.68 44.45) (xy 118.11 44.45)
-		)
-		(stroke
-			(width 0)
-			(type default)
-		)
-	)
-	(wire
-		(pts
 			(xy 34.29 190.5) (xy 27.94 190.5)
 		)
@@
 				(hide yes)
 			)
+		)
+	)
+	(global_label "SERVO_PWM"
+		(shape input)
+		(at 106.68 52.07 0)
+		(fields_autoplaced yes)
+		(effects
+			(font
+				(size 1.27 1.27)
+			)
+			(justify left)
+		)
+		(property "Intersheetrefs" "${INTERSHEET_REFS}"
+			(at 120.8532 52.07 0)
+			(effects
+				(font
+					(size 1.27 1.27)
+				)
+				(justify left)
+				(hide yes)
+			)
